File: schematic/WirelessPalaControl.sch (KiCad schematic (older format))
At the start: 20 parts, among them J1 6P6C, J2 MCU UART, Q1 BC847B, Q2 BC847B, U1 SI8621, U2 WeMos_mini

Commit message: Update schematic
Parts:
- C1, C2: value 100nF -> 100n; footprint Capacitors_SMD:C_0805_HandSoldering -> Capacitor_SMD:C_0805_2012Metric_Pad1.15x1.40mm_HandSolder
- D1, D3: footprint LEDs:LED_0805_HandSoldering -> LED_SMD:LED_0805_2012Metric_Pad1.15x1.40mm_HandSolder
- D2: footprint Diodes_SMD:D_SMA -> Diode_SMD:D_SMA
- J2: footprint Pin_Headers:Pin_Header_Straight_1x04_Pitch2.54mm -> Connector_PinHeader_2.54mm:PinHeader_1x04_P2.54mm_Vertical
- Q1, Q2: footprint TO_SOT_Packages_SMD:SOT-23_Handsoldering -> Package_TO_SOT_SMD:SOT-23_Handsoldering
- R1, R2, R3, R4, R5, R6, R7, R8: footprint Resistors_SMD:R_0805_HandSoldering -> Resistor_SMD:R_0805_2012Metric_Pad1.15x1.40mm_HandSolder
- U1: footprint Housings_SOIC:SOIC-8_3.9x4.9mm_Pitch1.27mm -> Package_SO:SOIC-8_3.9x4.9mm_P1.27mm
Changed lines of the file:
@@
 F 0 "Q2" H 1941 2696 50  0000 L CNN
 F 1 "BC847B" H 1941 2605 50  0000 L CNN
-F 2 "TO_SOT_Packages_SMD:SOT-23_Handsoldering" H 1950 2575 50  0001 L CIN
+F 2 "Package_TO_SOT_SMD:SOT-23_Handsoldering" H 1950 2575 50  0001 L CIN
 F 3 "http://www.infineon.com/dgdl/Infineon-BC847SERIES_BC848SERIES_BC849SERIES_BC850SERIES-DS-v01_01-en.pdf?fileId=db3a304314dca389011541d4630a1657" H 1750 2650 50  0001 L CNN
 	1    1750 2650
@@
 F 0 "J2" H 5980 2042 50  0000 L CNN
 F 1 "MCU UART" H 5980 1951 50  0000 L CNN
-F 2 "Pin_Headers:Pin_Header_Straight_1x04_Pitch2.54mm" H 5900 2050 50  0001 C CNN
+F 2 "Connector_PinHeader_2.54mm:PinHeader_1x04_P2.54mm_Vertical" H 5900 2050 50  0001 C CNN
 F 3 "~" H 5900 2050 50  0001 C CNN
 	1    5900 2050
@@
 F 0 "D1" H 1693 1545 50  0000 C CNN
 F 1 "RED" H 1693 1636 50  0000 C CNN
-F 2 "LEDs:LED_0805_HandSoldering" H 1700 1800 50  0001 C CNN
+F 2 "LED_SMD:LED_0805_2012Metric_Pad1.15x1.40mm_HandSolder" H 1700 1800 50  0001 C CNN
 F 3 "~" H 1700 1800 50  0001 C CNN
 	1    1700 1800
@@
 F 0 "R3" V 2250 2150 50  0000 C CNN
 F 1 "2K" V 2150 2150 50  0000 C CNN
-F 2 "Resistors_SMD:R_0805_HandSoldering" V 2080 2150 50  0001 C CNN
+F 2 "Resistor_SMD:R_0805_2012Metric_Pad1.15x1.40mm_HandSolder" V 2080 2150 50  0001 C CNN
 F 3 "~" H 2150 2150 50  0001 C CNN
 	1    2150 2150
@@
 F 0 "R2" V 3250 1950 50  0000 C CNN
 F 1 "220" V 3150 1950 50  0000 C CNN
-F 2 "Resistors_SMD:R_0805_HandSoldering" V 3080 1950 50  0001 C CNN
+F 2 "Resistor_SMD:R_0805_2012Metric_Pad1.15x1.40mm_HandSolder" V 3080 1950 50  0001 C CNN
 F 3 "~" H 3150 1950 50  0001 C CNN
 	1    3150 1950
@@
 F 0 "R7" V 5400 2250 50  0000 C CNN
 F 1 "220" V 5300 2250 50  0000 C CNN
-F 2 "Resistors_SMD:R_0805_HandSoldering" V 5230 2250 50  0001 C CNN
+F 2 "Resistor_SMD:R_0805_2012Metric_Pad1.15x1.40mm_HandSolder" V 5230 2250 50  0001 C CNN
 F 3 "~" H 5300 2250 50  0001 C CNN
 	1    5300 2250
@@
 F 0 "R6" V 5400 1950 50  0000 C CNN
 F 1 "1K" V 5300 1950 50  0000 C CNN
-F 2 "Resistors_SMD:R_0805_HandSoldering" V 5230 1950 50  0001 C CNN
+F 2 "Resistor_SMD:R_0805_2012Metric_Pad1.15x1.40mm_HandSolder" V 5230 1950 50  0001 C CNN
 F 3 "~" H 5300 1950 50  0001 C CNN
 	1    5300 1950
@@
 F 0 "D3" V 5139 2883 50  0000 R CNN
 F 1 "RED" V 5048 2883 50  0000 R CNN
-F 2 "LEDs:LED_0805_HandSoldering" H 5100 3000 50  0001 C CNN
+F 2 "LED_SMD:LED_0805_2012Metric_Pad1.15x1.40mm_HandSolder" H 5100 3000 50  0001 C CNN
 F 3 "~" H 5100 3000 50  0001 C CNN
 	1    5100 3000
@@
 P 3750 3300
 F 0 "C1" H 3865 3346 50  0000 L CNN
-F 1 "100nF" H 3865 3255 50  0000 L CNN
-F 2 "Capacitors_SMD:C_0805_HandSoldering" H 3788 3150 50  0001 C CNN
+F 1 "100n" H 3865 3255 50  0000 L CNN
+F 2 "Capacitor_SMD:C_0805_2012Metric_Pad1.15x1.40mm_HandSolder" H 3788 3150 50  0001 C CNN
 F 3 "~" H 3750 3300 50  0001 C CNN
 	1    3750 3300
@@
 P 4450 3300
 F 0 "C2" H 4565 3346 50  0000 L CNN
-F 1 "100nF" H 4565 3255 50  0000 L CNN
-F 2 "Capacitors_SMD:C_0805_HandSoldering" H 4488 3150 50  0001 C CNN
+F 1 "100n" H 4565 3255 50  0000 L CNN
+F 2 "Capacitor_SMD:C_0805_2012Metric_Pad1.15x1.40mm_HandSolder" H 4488 3150 50  0001 C CNN
 F 3 "~" H 4450 3300 50  0001 C CNN
 	1    4450 3300
@@
 F 0 "R8" H 5030 3304 50  0000 R CNN
 F 1 "1K" H 5030 3395 50  0000 R CNN
-F 2 "Resistors_SMD:R_0805_HandSoldering" V 5030 3350 50  0001 C CNN
+F 2 "Resistor_SMD:R_0805_2012Metric_Pad1.15x1.40mm_HandSolder" V 5030 3350 50  0001 C CNN
 F 3 "~" H 5100 3350 50  0001 C CNN
 	1    5100 3350
@@
 F 0 "D2" H 2500 2350 50  0000 C CNN
 F 1 "SS34" H 2500 2450 50  0000 C CNN
-F 2 "Diodes_SMD:D_SMA" H 2500 2250 50  0001 C CNN
+F 2 "Diode_SMD:D_SMA" H 2500 2250 50  0001 C CNN
 F 3 "~" H 2500 2250 50  0001 C CNN
 	1    2500 2250
@@
 F 0 "R1" V 3050 2150 50  0000 C CNN
 F 1 "1K" V 2950 2150 50  0000 C CNN
-F 2 "Resistors_SMD:R_0805_HandSoldering" V 2880 2150 50  0001 C CNN
+F 2 "Resistor_SMD:R_0805_2012Metric_Pad1.15x1.40mm_HandSolder" V 2880 2150 50  0001 C CNN
 F 3 "~" H 2950 2150 50  0001 C CNN
 	1    2950 2150
@@
 F 0 "U1" H 4150 2800 60  0000 L CNN
 F 1 "SI8621" H 4050 2700 60  0000 L CNN
-F 2 "Housings_SOIC:SOIC-8_3.9x4.9mm_Pitch1.27mm" H 4200 2100 50  0001 C CNN
+F 2 "Package_SO:SOIC-8_3.9x4.9mm_P1.27mm" H 4200 2100 50  0001 C CNN
 F 3 "" H 4200 2100 50  0001 C CNN
 	1    4200 2100
@@
 F 0 "R5" V 3000 2800 50  0000 C CNN
 F 1 "2K" V 2900 2800 50  0000 C CNN
-F 2 "Resistors_SMD:R_0805_HandSoldering" V 2830 2800 50  0001 C CNN
+F 2 "Resistor_SMD:R_0805_2012Metric_Pad1.15x1.40mm_HandSolder" V 2830 2800 50  0001 C CNN
 F 3 "~" H 2900 2800 50  0001 C CNN
 	1    2900 2800
@@
 F 0 "R4" V 3150 3050 50  0000 C CNN
 F 1 "2K" V 3250 3050 50  0000 C CNN
-F 2 "Resistors_SMD:R_0805_HandSoldering" V 3180 3050 50  0001 C CNN
+F 2 "Resistor_SMD:R_0805_2012Metric_Pad1.15x1.40mm_HandSolder" V 3180 3050 50  0001 C CNN
 F 3 "~" H 3250 3050 50  0001 C CNN
 	1    3250 3050
@@
 F 0 "Q1" H 3191 3296 50  0000 L CNN
 F 1 "BC847B" H 3191 3205 50  0000 L CNN
-F 2 "TO_SOT_Packages_SMD:SOT-23_Handsoldering" H 3200 3175 50  0001 L CIN
+F 2 "Package_TO_SOT_SMD:SOT-23_Handsoldering" H 3200 3175 50  0001 L CIN
 F 3 "http://www.infineon.com/dgdl/Infineon-BC847SERIES_BC848SERIES_BC849SERIES_BC850SERIES-DS-v01_01-en.pdf?fileId=db3a304314dca389011541d4630a1657" H 3000 3250 50  0001 L CNN
 	1    3000 3250
